File: piezo_amplifier/piezo_amplifier.sch (KiCad schematic (older format))
At the start: 38 parts, among them J1 Conn_01x02_Female, J2 Conn_01x02_Female, J3 Conn_01x02_Female, J4 Conn_01x02_Female, J5 Conn_01x02_Female, J6 Conn_01x02_Female, U1 LMV324, U2 TLV76033DBZT, U3 TLP185

Commit message: PCB and schematics files finished, ready for release.
Parts:
- removed J2: Conn_01x02_Female, Connector_JST:JST_XH_S02B-XH-A_1x02_P2.50mm_Horizontal, symbol Connector:Conn_01x02_Female
- added C9: 1uF, Capacitor_SMD:C_0603_1608Metric, symbol Device:C
- J1, J3, J4, J5, J6: footprint Connector_JST:JST_XH_S02B-XH-A_1x02_P2.50mm_Horizontal -> Connector_JST:JST_XH_S2B-XH-A_1x02_P2.50mm_Horizontal
- POT1, POT2: footprint digikey-footprints:Trimpot_3.8mmx3.6mm_TC33X-2-103E -> Potentiometer_SMD:Potentiometer_Bourns_TC33X_Vertical
- TP1, TP2, TP3, TP4, TP5, TP6: footprint (none) -> TestPoint:TestPoint_Loop_D1.80mm_Drill1.0mm_Beaded
- U2: footprint digikey-footprints:SOT-23-3 -> Package_TO_SOT_SMD:SOT-23
Connections:
- wire segments 110 -> 107
Other:
- note added: "Note: \nPlace decoupling capacitor \nclose to the supply pins\n"
- note removed: "From PCB hotend fan output"
- note removed: "Note: Place decoupling capacitor close to the supply pins\n"
- note removed: "To hotend fan"
- moved on the sheet: C1, C2, C3, C5, C6, D1, D3, J1, R7, TP4, U1A, U1C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

Commit message: Version V2.0 released
Parts:
- removed J1, J3, J4, J5, J6: Conn_01x02_Female, Connector_JST:JST_XH_S2B-XH-A_1x02_P2.50mm_Horizontal, symbol Connector:Conn_01x02_Female
- removed U1: LMV324, Package_SO:SOIC-14_3.9x8.7mm_P1.27mm, symbol Amplifier_Operational:LMV324
- added J1, J3, J4, J5, J6: S2B-XH-A-1, Connector_JST:JST_XH_S2B-XH-A_1x02_P2.50mm_Horizontal, symbol CON:S2B-XH-A-1
- added U1: LMV324, Package_SO:SOIC-14_3.9x8.7mm_P1.27mm, symbol IC_Analog:LMV324
- C1: Comment (none) -> 35V, 10%; Description (none) -> 35V, 10%; Populate (none) -> 1
- C2, C3, C4, C5, C7, C8, C9: Comment (none) -> 6.3V, 10%; Description (none) -> 6.3V, 10%; Populate (none) -> 1
- C6: Comment (none) -> 6.3V, 10%; Populate (none) -> 1
- D1: Comment (none) -> Red LED; Populate (none) -> 1
- D2, R10, R9: Populate (none) -> 1
- D3: Comment (none) -> Green LED; Populate (none) -> 1
- POT1: value 10K -> 10K_SMD; footprint Potentiometer_SMD:Potentiometer_Bourns_TC33X_Vertical -> digikey-footprints:Trimpot_3.8mmx3.6mm_TC33X-2-103E; symbol piezo_amplifier-rescue:TC33X-2-103E-dk_Trimmer-Potentiometers -> Resistor_POT:10K_SMD; Populate (none) -> 1
- POT2: value TC33X-2-103E -> 10K_SMD; footprint Potentiometer_SMD:Potentiometer_Bourns_TC33X_Vertical -> digikey-footprints:Trimpot_3.8mmx3.6mm_TC33X-2-103E; symbol piezo_amplifier-rescue:TC33X-2-103E-dk_Trimmer-Potentiometers -> Resistor_POT:10K_SMD; Populate (none) -> 1
- R1, R3, R4, R5, R6: Comment (none) -> 1%; Populate (none) -> 1
- R2: Comment  (none) -> 1%; Populate (none) -> 1
- R7: Comment (none) -> 5%; Populate (none) -> 1
- R8: Comment (none) -> 1%; Description (none) -> 1%; Populate (none) -> 0
- TP1, TP2, TP3, TP5, TP6, U3: Populate (none) -> 0
- U2: value TLV76033DBZT -> TLV76033; footprint Package_TO_SOT_SMD:SOT-23 -> digikey-footprints:SOT-23-3; symbol piezo_amplifier-rescue:TLV76033DBZT-OD_Analog -> IC_Analog:TLV76033; Populate (none) -> 1
Other:
- moved on the sheet: D1

Commit message: Piezo amplifier V2.0 released. Updated with the new library convention to show not installed components and standardizing fields.
Parts:
- removed C1, C5, C9: 1uF, Capacitor_SMD:C_0603_1608Metric, symbol Device:C
- removed C2, C3, C4, C7, C8: 22nF, Capacitor_SMD:C_0603_1608Metric, symbol Device:C
- removed C6: 2nF, Capacitor_SMD:C_0603_1608Metric, symbol Device:C
- removed R1, R2, R5, R6: 10K, Resistor_SMD:R_0603_1608Metric, symbol Device:R
- removed R10, R9: 0R, Resistor_SMD:R_0603_1608Metric, symbol Device:R
- removed R3, R7: 330, Resistor_SMD:R_0603_1608Metric, symbol Device:R
- removed R4: 20K, Resistor_SMD:R_0603_1608Metric, symbol Device:R
- removed R8: 330R, Resistor_SMD:R_0603_1608Metric, symbol Device:R
- added C1, C5, C9: 1uF, Capacitor_SMD:C_0603_1608Metric_Pad1.05x0.95mm_HandSolder, symbol Capacitor_Ceramic_SMD_0603:1uF
- added C2, C3, C4, C6, C7, C8: 22nF, Capacitor_SMD:C_0603_1608Metric_Pad1.05x0.95mm_HandSolder, symbol Capacitor_Ceramic_SMD_0603:22nF
- added R1, R2, R5, R6: 10K, Resistor_SMD:R_0603_1608Metric, symbol Resistor_SMD_0603:10K
- added R10, R9: 0R, Resistor_SMD:R_0603_1608Metric, symbol Resistor_SMD_0603:0R
- added R3, R7, R8: 330R, Resistor_SMD:R_0603_1608Metric, symbol Resistor_SMD_0603:330R
- added R4: 20K, Resistor_SMD:R_0603_1608Metric, symbol Resistor_SMD_0603:20K
- D1: symbol Device:LED -> OPTO_LED_0603:Green
- D3: symbol Device:LED -> OPTO_LED_0603:Green; Comment Green LED -> (none); Description (none) -> LED Green 20mA 2V; Generic (none) -> 0; Installed (none) -> NI; MPN (none) -> 150060VS75000; Manufacturer (none) -> Würth Elektronik; Populate 1 -> (none)
- POT1, POT2: value 10K_SMD -> 10K; symbol Resistor_POT:10K_SMD -> Resistor_POT:10K; Description TRIMMER 10K OHM 0.1W J LEAD TOP -> TRIMMER 10K OHM 0.1W J LEAD TOP SMD; Generic (none) -> 1
- TP1, TP2, TP3, TP5, TP6: Installed (none) -> NU; Populate 0 -> (none)
- TP4, U1: Installed (none) -> NI
- U1: Description LMV3xxLow-Voltage Rail-to-Rail Output Operational Amplifier -> IC Opamp R-TO-R Low voltage SOIC14; Generic (none) -> 0; Installed (none) -> NI; Manufacturer (none) -> Texas Instruments
- U1: Installed (none) -> NI; Populate 1 -> (none)
- U2: footprint digikey-footprints:SOT-23-3 -> Package_TO_SOT_SMD:SOT-23; Generic (none) -> 0; Installed (none) -> NI
- U3: Description OPhotocoupler, GaAs Ired & Photo−Transistor -> Optocoupler 80V SOIC 4; Generic (none) -> 0; Installed (none) -> NU; MPN TLP185(GR-TPL,E(O -> TLP185(GR,E(O; Populate 0 -> (none)
Other:
- note added: "-The TVS diode protects the input from overvoltage\n-The RC implements a low pass filter in the case \nit is needed, but C7 is not populated by default."
- note added: "The otput can be isolated using \nan optocoupler.This is optional \nbut helps preventing ground loops.\n\nBy default R9 and R10 are installed, U3 is uninstalled.\n"
- note removed: "-The TVS diode protects the input from overvoltage\n-The RC implements a low pass filter in the case \nit is needed, but C is not populated by default."
- note removed: "The otput can be isolated using \nan optocoupler.This is optional \nbut helps preventing ground loops.\n"

Commit message: fixup! fixup! Piezo amplifier V2.0 released. Updated with the new library convention to show not installed components and standardizing fields.
Parts:
- R10, R9: Installed NU -> NI
Changed lines of the file:
@@
 F 5 "1" H 9000 4000 50  0001 C CNN "Populate"
 F 6 "1" H 9000 4000 50  0001 C CNN "Generic"
-F 7 "NU" H 9000 4000 50  0001 C CNN "Installed"
+F 7 "NI" H 9000 4000 50  0001 C CNN "Installed"
 	1    9000 4000
 	0    1    1    0
@@
 F 5 "1" H 9000 4750 50  0001 C CNN "Populate"
 F 6 "1" H 9000 4750 50  0001 C CNN "Generic"
-F 7 "NU" H 9000 4750 50  0001 C CNN "Installed"
+F 7 "NI" H 9000 4750 50  0001 C CNN "Installed"
 	1    9000 4750
 	0    1    1    0
